File: Lifedatalink_v1_revB.kicad_sch (KiCad schematic)
At the start: 91 parts

Commit message: Change linear regulators for more current capacity
Parts:
- removed C31: (no value), symbol Device:C
- removed R17, R18, R19, R20, R21: (no value), symbol Device:R
- removed U2: (no value), symbol dk_PMIC-Voltage-Regulators-Linear:LP5907MFX-3_3_NOPB
- removed U7: (no value), symbol Regulator_Linear:LP5907MFX-1.8
- removed U9: (no value), symbol Interface:PCA9306
- added U2: NCP167BMX330TBG, REG_NCP167BMX330TBG, symbol NCP167BMX330TBG:NCP167BMX330TBG
- added U7: NCP167AMX180TBG, REG_NCP167BMX330TBG, symbol NCP167BMX330TBG:NCP167BMX330TBG
- C1, C10, C11, C12, C13, C14, C15, C16, C17, C18, C19, C2, C20, C21, C22, C23, C24, C27, C28, C29, C30, C5, C6, C7, C8, C9, D1, D2, J1, J10, J11, J12, J13, J14, J15, J16, J17, J18, J19, J2, J20, J3, J4, J5, J6, J7, J8, J9, MIC1, MIC2, R1, R10, R11, R12, R13, R14, R15, R16, R2, R22, R5, R6, R7, R8, R9, SW1, U1, U3, U4, U5, U6, U8, Y1: value (none) -> ~
- C25, C26, C3, C4: value (none) -> 1u
- D3: value (none) -> MBR0540T1G
- F1: value (none) -> 0603L075SLYR
- Q1: value (none) -> CSD23280F3
- R3: value (none) -> 2K
- R4: value (none) -> 100K
Connections:
- net +1V8: now also U7.1 (OUT)
- net +3V3: no longer C25.2, C4.2, R5.2
- net +5V: no longer C6.2, D1.6 (VBUS), D3.2, J1.A4 (VBUS), J1.A9 (VBUS), J1.B4 (VBUS), J1.B9 (VBUS), Q1.1 (G), R4.2, U4.4 (VDD)
- net GND: now also U2.2 (GND), U2.5 (EXP), U7.2 (GND), U7.5 (EXP); no longer J1.S1 (SHIELD), J1.S2 (SHIELD), J1.S3 (SHIELD), J1.S4 (SHIELD)
- net VIN: now also U2.3 (EN), U2.4 (IN)
- new net: J1.S1 (SHIELD), J1.S2 (SHIELD), J1.S3 (SHIELD), J1.S4 (SHIELD)
- new net +3.3V: C25.2, C4.2, R5.2, U2.1 (OUT), U7.3 (EN), U7.4 (IN)
- new net VBUS: C6.2, D1.6 (VBUS), D3.2, J1.A4 (VBUS), J1.A9 (VBUS), J1.B4 (VBUS), J1.B9 (VBUS), Q1.1 (G), R4.2, U4.4 (VDD)
- no-connect marks 0 -> 14
Other:
- note added: "Load sharing"
- note removed: "I2C LEVEL SHIFTER"
- moved on the sheet: C25, C26, C4

Commit message: Add values to ADS and BLE
Parts:
- removed R15, R16: ~, symbol Device:R
- added C31: 0.1u, symbol Device:C
- C1, C2: value ~ -> 12p
- C10: value ~ -> 10u
- C11, C12, C23, C8: value ~ -> 1u
- C13, C14: value ~ -> 47n
- C15, C16, C18, C20: value ~ -> 2.2n
- C17, C19, C22, C5, C9: value ~ -> 0.1u
- C6, C7: value ~ -> 4.7u
- D2: value ~ -> APA-102-2020-256-8
- R1, R2: value ~ -> 1K
- R10, R5, R6, R9: value ~ -> 10M
- R3: value 2K -> 10K
- R7, R8: value ~ -> 40.2k
- U1: value ~ -> BL654
- U3: value ~ -> ADS1292
- Y1: value ~ -> 32.768 kHz
Connections:
- net +5V is gone; now on net VBUS: U1.24 (VBUS)
- net +3.3V: now also C22.2, C23.2, C5.2, C8.2, R1.2, U1.25 (VDD_HV), U1.31 (VDD), U3.12 (AVDD), U3.23 (DVDD), C31.2
- net +3V3: no longer C22.2, C23.2, C5.2, C8.2, U1.25 (VDD_HV), U1.31 (VDD), U3.12 (AVDD), U3.23 (DVDD)
- net +BATT: no longer R1.2
- net GND: now also C31.1
- net ADS_GPIO2: now reaches U3.25 (GPIO2/RCLK2)
- net ADS_GPIO1: now reaches U3.26 (GPIO1/RCLK1)
Other:
- moved on the sheet: C10, C12, C13, C14, C9, R1, R2
